File: pcb/Clay ibm/Clay ibm.kicad_sch (KiCad schematic)
At the start: 1 part

Commit message: stuff
Parts:
- added D? (x4): D_Small, symbol Device:D_Small
- added D?: SK6812, LED_SMD:LED_SK6812_PLCC4_5.0x5.0mm_P3.2mm, symbol LED:SK6812
- added MX? (x4): MX-NoLED, symbol MX_Alps_Hybrid:MX-NoLED
Connections:
- net C1: now also MX?.1 (COL), MX?.1 (COL)
- net C2: now also MX?.1 (COL), MX?.1 (COL)
- net R1: now also D?.1 (K), D?.1 (K)
- net R2: now also D?.1 (K), D?.1 (K)
- new net: D?.2 (A), MX?.2 (ROW) (x4)
Other:
- moved on the sheet: U?
